File: schematics/kiCad/blinky-cube.kicad_pcb (KiCad board)
At the start: 2 copper layers, 59 x 53 mm, 14 parts, among them J1 Screw_Terminal_01x02, J2 Screw_Terminal_01x03, J3 Screw_Terminal_01x03, SW1 SW_Push, U1 Pico

Commit message: schematic in DIN mode 3 format
Parts:
- removed ? (x2): , 
- added J4: Screw_Terminal_01x03, TerminalBlock:TerminalBlock_bornier-3_P5.08mm, F.Cu at (181.9, 95.1)
- added R5: 10k, Resistor_SMD:R_1206_3216Metric_Pad1.30x1.75mm_HandSolder, B.Cu at (112.5, 86.5)
- D1, J2, J3, SW1: moved to F.Cu
- J1: value Screw_Terminal_01x02 -> Screw_Terminal_01x03; footprint TerminalBlock:TerminalBlock_bornier-2_P5.08mm -> TerminalBlock:TerminalBlock_bornier-3_P5.08mm; moved to F.Cu
- moved D1 87.4 mm to (181.9, 53.2), turned to -90 degrees
- moved R1 85.4 mm to (173.5, 53.2), turned to 0 degrees
- moved SW1 71.3 mm to (184.2, 61.4), turned to -90 degrees
- moved R2 66.5 mm to (173.6, 61.3), turned to 180 degrees
- moved J3 54.9 mm to (105.5, 69.7), turned to -90 degrees
- moved R4 52.3 mm to (112.5, 71.0), turned to 90 degrees
- moved R3 47.2 mm to (112.5, 56.0), turned to 90 degrees
- moved G*** 45.2 mm to (147.0, 57.0)
- moved C1 39.1 mm to (163.8, 90.2), turned to 180 degrees
- moved U1 37.4 mm to (143.8, 74.9), turned to -90 degrees
- moved J1 37.0 mm to (105.5, 54.5), turned to -90 degrees
- moved J2 33.3 mm to (105.5, 85.0), turned to -90 degrees
Connections:
- C1 pad 1: Net-(C1-Pad1) -> Net-(J4-Pin_1)
- D1 pad 2: Net-(D1-Pad2) -> Net-(D1-A)
- J1 pad 1: Net-(C1-Pad1) -> Net-(J1-Pin_1)
- J1 pad 2: GND -> Net-(J1-Pin_2)
- J2 pad 1: Net-(SW1-Pad1) -> Net-(J2-Pin_1)
- J2 pad 2: Net-(U1-Pad24) -> Net-(J2-Pin_2)
- J3 pad 1: Net-(SW1-Pad1) -> Net-(J3-Pin_1)
- J3 pad 2: Net-(U1-Pad21) -> Net-(J3-Pin_2)
- R2 pad 1: Net-(R2-Pad1) -> Net-(U1-GPIO3)
- R3 pad 1: Net-(U1-Pad24) -> Net-(J1-Pin_2)
- R3 pad 2: Net-(SW1-Pad1) -> Net-(J1-Pin_1)
- R4 pad 1: Net-(U1-Pad21) -> Net-(J3-Pin_2)
- R4 pad 2: Net-(SW1-Pad1) -> Net-(J3-Pin_1)
- SW1 pad 1: Net-(SW1-Pad1) -> Net-(U1-3V3)
- SW1 pad 2: Net-(R2-Pad1) -> Net-(U1-GPIO3)
- U1 pad 15: Net-(D1-Pad2) -> Net-(J1-Pin_1)
- U1 pad 16: unconnected-(U1-Pad16) -> Net-(J1-Pin_2)
- U1 pad 19: unconnected-(U1-Pad19) -> Net-(J3-Pin_1)
- U1 pad 20: Net-(R2-Pad1) -> Net-(J3-Pin_2)
- U1 pad 21: Net-(U1-Pad21) -> Net-(J2-Pin_1)
- U1 pad 22: unconnected-(U1-Pad22) -> Net-(J2-Pin_2)
- U1 pad 24: Net-(U1-Pad24) -> unconnected-(U1-GPIO18-Pad24)
- U1 pad 36: Net-(SW1-Pad1) -> Net-(U1-3V3)
- U1 pad 39: unconnected-(U1-Pad39) -> Net-(J4-Pin_1)
- U1 pad 4: unconnected-(U1-Pad4) -> Net-(D1-A)
- U1 pad 40: Net-(C1-Pad1) -> unconnected-(U1-VBUS-Pad40)
- U1 pad 5: unconnected-(U1-Pad5) -> Net-(U1-GPIO3)
Routing:
- net Net-(SW1-Pad1): track 143.4 -> 0.00 mm
- net Net-(U1-3V3): track 0.00 -> 40.4 mm
- net Net-(U1-GPIO3): track 0.00 -> 39.2 mm
- net Net-(J1-Pin_1): track 0.00 -> 35.5 mm
- net Net-(U1-Pad24): track 34.9 -> 0.00 mm
- net Net-(J1-Pin_2): track 0.00 -> 31.0 mm
- net Net-(J4-Pin_1): track 0.00 -> 28.0 mm
- net Net-(D1-A): track 0.00 -> 25.8 mm
- net Net-(J3-Pin_1): track 0.00 -> 25.5 mm
- net Net-(U1-Pad21): track 23.6 -> 0.00 mm
- net Net-(D1-Pad2): track 21.7 -> 0.00 mm
- net Net-(J3-Pin_2): track 0.00 -> 20.4 mm
- net Net-(J2-Pin_2): track 0.00 -> 20.3 mm
- net Net-(C1-Pad1): track 17.7 -> 0.00 mm
- net Net-(R2-Pad1): track 17.5 -> 0.00 mm
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Other:
- board size 59 x 53 mm -> 86.6 x 49.7 mm
- board text added: "blinky-DS18B20-p-cube v2.0"

Commit message: first commit
Parts:
- removed R3, R4, R5: 10k, Resistor_SMD:R_1206_3216Metric_Pad1.30x1.75mm_HandSolder
- added C2: 0.1uF, Capacitor_SMD:C_1206_3216Metric_Pad1.33x1.80mm_HandSolder, B.Cu at (109.5, 90.1)
- added C3: 0.1uF, Capacitor_SMD:C_1206_3216Metric_Pad1.33x1.80mm_HandSolder, B.Cu at (116.4, 82.6)
- added C4: 0.1uF, Capacitor_SMD:C_1206_3216Metric_Pad1.33x1.80mm_HandSolder, B.Cu at (116.3, 67.2)
- added C5: 0.1uF, Capacitor_SMD:C_1206_3216Metric_Pad1.33x1.80mm_HandSolder, B.Cu at (109.7, 74.9)
- added C6: 0.1uF, Capacitor_SMD:C_1206_3216Metric_Pad1.33x1.80mm_HandSolder, B.Cu at (117.6, 54.0)
- added C7: 0.1uF, Capacitor_SMD:C_1206_3216Metric_Pad1.33x1.80mm_HandSolder, B.Cu at (109.4, 59.4)
- added FB1: FerriteBead, Inductor_SMD:L_1206_3216Metric_Pad1.42x1.75mm_HandSolder, B.Cu at (110.9, 95.1)
- added FB2: FerriteBead, Inductor_SMD:L_1206_3216Metric_Pad1.42x1.75mm_HandSolder, B.Cu at (110.8, 85.0)
- added FB3: FerriteBead, Inductor_SMD:L_1206_3216Metric_Pad1.42x1.75mm_HandSolder, B.Cu at (110.8, 79.8)
- added FB4: FerriteBead, Inductor_SMD:L_1206_3216Metric_Pad1.42x1.75mm_HandSolder, B.Cu at (110.8, 69.7)
- added FB5: FerriteBead, Inductor_SMD:L_1206_3216Metric_Pad1.42x1.75mm_HandSolder, B.Cu at (110.7, 64.6)
- added FB6: FerriteBead, Inductor_SMD:L_1206_3216Metric_Pad1.42x1.75mm_HandSolder, B.Cu at (110.8, 54.5)
- added U2: MAX31855KASA+, LM358AD:SOIC127P600X175-8N, B.Cu at (116.2, 90.0)
- added U3: MAX31855KASA+, LM358AD:SOIC127P600X175-8N, B.Cu at (116.2, 74.8)
- added U4: MAX31855KASA+, LM358AD:SOIC127P600X175-8N, B.Cu at (116.2, 59.4)
- moved C1 6.60 mm to (170.4, 90.2)
- moved U1 6.24 mm to (150.0, 74.8)
Connections:
- net Net-(U1-3V3) renamed /3V3
- J1 pad 2: Net-(J1-Pin_2) -> GND
- J1 pad 3: GND -> Net-(J1-Pin_3)
- J2 pad 2: Net-(J2-Pin_2) -> GND
- J2 pad 3: GND -> Net-(J2-Pin_3)
- J3 pad 2: Net-(J3-Pin_2) -> GND
- J3 pad 3: GND -> Net-(J3-Pin_3)
- U1 pad 15: Net-(J1-Pin_1) -> unconnected-(U1-GPIO11-Pad15)
- U1 pad 16: Net-(J1-Pin_2) -> unconnected-(U1-GPIO12-Pad16)
- U1 pad 19: Net-(J3-Pin_1) -> unconnected-(U1-GPIO14-Pad19)
- U1 pad 20: Net-(J3-Pin_2) -> unconnected-(U1-GPIO15-Pad20)
- U1 pad 21: Net-(J2-Pin_1) -> /SPIO_RX
- U1 pad 22: Net-(J2-Pin_2) -> /SPIO_CS4
- U1 pad 24: unconnected-(U1-GPIO18-Pad24) -> /SPIO_CLK
- U1 pad 26: unconnected-(U1-GPIO20-Pad26) -> /SPIO_CS3
- U1 pad 27: unconnected-(U1-GPIO21-Pad27) -> /SPIO_CS2
Routing:
- net /3V3: track 40.4 -> 158.6 mm, vias 0 -> 3
- net /SPIO_CS4: track 0.00 -> 79.4 mm, vias 0 -> 1
- net /SPIO_CLK: track 0.00 -> 53.1 mm, vias 0 -> 3
- net /SPIO_RX: track 0.00 -> 50.5 mm, vias 0 -> 3
- net /SPIO_CS3: track 0.00 -> 34.3 mm, vias 0 -> 1
- net Net-(J1-Pin_1): track 35.5 -> 3.78 mm
- net Net-(J1-Pin_2): track 31.0 -> 0.00 mm
- net /SPIO_CS2: track 0.00 -> 26.7 mm
- net Net-(J3-Pin_1): track 25.5 -> 3.82 mm
- net Net-(J3-Pin_2): track 20.4 -> 0.00 mm
- net Net-(J2-Pin_2): track 20.3 -> 0.00 mm
- net Net-(J2-Pin_1): track 14.6 -> 3.83 mm
- net Net-(U4-T-): track 0.00 -> 9.35 mm
- net Net-(U4-T+): track 0.00 -> 9.10 mm
- net Net-(U2-T-): track 0.00 -> 9.06 mm
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Other:
- board text added: "blinky-thermo-couple-p-cube v2.0"
- board text removed: "blinky-DS18B20-p-cube v2.0"
