File: schematics/kiCad/blinky-cube.kicad_sch (KiCad schematic)
At the start: 11 parts, among them J1 Screw_Terminal_01x02, J2 Screw_Terminal_01x03, J3 Screw_Terminal_01x03, SW1 SW_Push, U1 Pico

Commit message: schematic in DIN mode 3 format
Parts:
- removed J1: Screw_Terminal_01x02, TerminalBlock:TerminalBlock_bornier-2_P5.08mm, symbol Connector:Screw_Terminal_01x02
- added J1, J4: Screw_Terminal_01x03, TerminalBlock:TerminalBlock_bornier-3_P5.08mm, symbol Connector:Screw_Terminal_01x03
- added R5: 10k, Resistor_SMD:R_1206_3216Metric_Pad1.30x1.75mm_HandSolder, symbol Device:R
Connections:
- net GND: now also J1.3 (Pin_3), J4.3 (Pin_3)
- net at R2.1, SW1.2: now also U1.5 (GPIO3); no longer U1.20 (GPIO15)
- net at C1.1: now also U1.39 (VSYS), J4.1 (Pin_1), J4.2 (Pin_2); no longer U1.40 (VBUS)
- net at U1.15 (GPIO11): now also R3.2, J1.1 (Pin_1); no longer D1.2 (A)
- net at U1.16 (GPIO12): now also R3.1, J1.2 (Pin_2)
- net at U1.19 (GPIO14): now also J3.1 (Pin_1), R4.2
- net at J3.2 (Pin_2), R4.1: now also U1.20 (GPIO15); no longer U1.21 (GPIO16)
- net at U1.22 (GPIO17): now also J2.2 (Pin_2), R5.1
- net at U1.4 (GPIO2): now also D1.2 (A)
- new net: J2.1 (Pin_1), R5.2, U1.21 (GPIO16)
- new net: SW1.1, U1.36 (3V3)
- now unconnected: U1.24 (GPIO18)
- no-connect marks 26 -> 22
Other:
- note added: "blinky-DS18B20-p-cube v2.0"
- moved on the sheet: C1, D1, R1, R2, SW1

Commit message: first commit
Parts:
- removed R3, R4, R5: 10k, Resistor_SMD:R_1206_3216Metric_Pad1.30x1.75mm_HandSolder, symbol Device:R
- added C2, C3, C4, C5, C6, C7: 0.1uF, Capacitor_SMD:C_1206_3216Metric_Pad1.33x1.80mm_HandSolder, symbol Device:C
- added FB1, FB2, FB3, FB4, FB5, FB6: FerriteBead, Inductor_SMD:L_1206_3216Metric_Pad1.42x1.75mm_HandSolder, symbol Device:FerriteBead
- added U2, U3, U4: MAX31855KASA+, SOIC127P600X175-8N, symbol MAX31855KASA_:MAX31855KASA+
Connections:
- net GND: now also J1.2 (Pin_2), J2.2 (Pin_2), J3.2 (Pin_2), C3.2, C4.2, C6.2, U2.1 (GND), U3.1 (GND), U4.1 (GND); no longer J1.3 (Pin_3), J2.3 (Pin_3), J3.3 (Pin_3)
- net at U1.15 (GPIO11): no longer J1.1 (Pin_1)
- net at U1.16 (GPIO12): no longer J1.2 (Pin_2)
- net at U1.19 (GPIO14): no longer J3.1 (Pin_1)
- net at U1.20 (GPIO15): no longer J3.2 (Pin_2)
- net at J2.1 (Pin_1): now also FB2.2; no longer U1.21 (GPIO16)
- net SPIO_CS4: now reaches U1.22 (GPIO17)
- net SPIO_CS4: now also U4.6 (~{CS}); no longer J2.2 (Pin_2)
- net SPIO_CLK: now reaches U1.24 (GPIO18)
- net SPIO_CLK: now also U2.5 (SCK), U3.5 (SCK), U4.5 (SCK)
- net SPIO_CS3: now reaches U1.26 (GPIO20)
- net SPIO_CS3: now also U3.6 (~{CS})
- net SPIO_CS2: now reaches U1.27 (GPIO21)
- net SPIO_CS2: now also U2.6 (~{CS})
- net 3V3: now reaches SW1.1, U1.36 (3V3)
- net 3V3: now also C3.1, C4.1, C6.1, U2.4 (VCC), U3.4 (VCC), U4.4 (VCC)
- new net: C7.1, FB5.1, U4.2 (T-)
- new net: C7.2, FB6.1, U4.3 (T+)
- new net: FB6.2, J1.1 (Pin_1)
- new net: C5.2, FB4.1, U3.3 (T+)
- new net: FB4.2, J3.1 (Pin_1)
- new net: C5.1, FB3.1, U3.2 (T-)
- new net: C2.1, FB1.1, U2.2 (T-)
- new net: C2.2, FB2.1, U2.3 (T+)
- new net: FB3.2, J3.3 (Pin_3)
- new net: FB5.2, J1.3 (Pin_3)
- new net: FB1.2, J2.3 (Pin_3)
- new net SPIO_RX: U1.21 (GPIO16), U2.7 (SO), U3.7 (SO), U4.7 (SO)
- no-connect marks 22 -> 23
Other:
- note added: "blinky-thermo-couple-p-cube v2.0"
- note removed: "blinky-DS18B20-p-cube v2.0"
- moved on the sheet: J1, J2, J3
